Commit message: Add additional links and joints to the skyentific_robot URDF for enhanced functionality

File: install/robot_description/share/robot_description/urdf/skyentific_robot.urdf.xacro (robot description, xacro)
@@ -44,4 +44,109 @@
         </collision>
     </link>
+    <link name="link_2">
+        <visual>
+            <origin xyz="0 0 0" rpy="0 0 0" />
+            <geometry>
+                <mesh filename="file://$(find robot_description)/meshes/link_2.stl"
+                    scale="0.001 0.001 0.001" />
+            </geometry>
+            <material name="grey" />
+        </visual>
+        <collision>
+            <origin xyz="0.225 0 0 " rpy="0 0 0" />
+            <geometry>
+                <cylinder radius="0.07" length="0.1" />
+            </geometry>
+        </collision>
+    </link>
+    <link name="link_3">
+        <visual>
+            <origin xyz="0 0 0" rpy="0 0 0" />
+            <geometry>
+                <mesh filename="file://$(find
+robot_description)/meshes/link_3.stl"
+                    scale="0.001 0.001 0.001" />
+            </geometry>
+            <material name="grey" />
+        </visual>
+        <collision>
+            <origin xyz="0.2 0 0" rpy="0 0 0" />
+            <geometry>
+                <cylinder radius="0.055" length="0.1" />
+            </geometry>
+        </collision>
+    </link>
+    <link name="link_4">
+        <visual>
+            <origin xyz="0 0 0" rpy="0 0 0" />
+            <geometry>
+                <mesh filename="file://$(find
+robot_description)/meshes/link_4.stl"
+                    scale="0.001 0.001 0.001" />
+            </geometry>
+            <material name="grey" />
+        </visual>
+        <collision>
+            <origin xyz="0.1 0 0" rpy="0 1.57 0" />
+            <geometry>
+                <cylinder radius="0.055"
+                    length="0.06" />
+            </geometry>
+        </collision>
+    </link>
+    <link name="link_5">
+        <visual>
+            <origin xyz="0 0 0" rpy="0 0 0" />
+            <geometry>
+                <mesh filename="file://$(find
+robot_description)/meshes/link_5_gripper.stl"
+                    scale="0.001 0.001 0.001" />
+            </geometry>
+            <material name="grey" />
+        </visual>
+        <collision>
+            <origin xyz="0 0 0" rpy="1.57 0 0" />
+            <geometry>
+                <cylinder radius="0.055"
+                    length="0.01" />
+            </geometry>
+        </collision>
+    </link>
+    <link name="gripper_right">
+        <visual>
+            <origin xyz="0 0 0" rpy="0 0 0" />
+            <geometry>
+                <mesh filename="file://$(find
+robot_description)/meshes/rightjaw.stl"
+                    scale="0.001 0.001 0.001" />
+            </geometry>
+            <material name="red" />
+        </visual>
+        <collision>
+            <origin xyz="0.01 0.025 0.045" rpy="0 0 0" />
+            <geometry>
+                <cylinder radius="0.0125"
+                    length="0.04" />
+            </geometry>
+        </collision>
+    </link>
+    <link name="gripper_left">
+        <visual>
+            <origin xyz="0 0 0" rpy="0 0 0" />
+            <geometry>
+                <mesh filename="file://$(find
+robot_description)/meshes/leftjaw.stl"
+                    scale="0.001 0.001 0.001" />
+            </geometry>
+            <material name="red" />
+        </visual>
+        <collision>
+            <origin xyz="0.01 -0.025 0.045" rpy="0 0 0" />
+            <geometry>
+                <cylinder radius="0.0125"
+                    length="0.04" />
+            </geometry>
+        </collision>
+    </link>
     <joint name="joint_1" type="revolute">
         <parent link="base_link" />
@@ -52,3 +157,52 @@
             lower="-3.14" upper="3.14" />
     </joint>
+    <joint name="joint_2" type="revolute">
+        <parent link="link_1" />
+        <child link="link_2" />
+        <origin xyz="0 0 0.150" rpy="0 -1.57 1.57 " />
+        <axis xyz="0 0 1" />
+        <limit effort="1000.0" velocity="100.0"
+            lower="-2.51" upper="2.51" />
+    </joint>
+    <joint name="joint_3" type="revolute">
+        <parent link="link_2" />
+        <child link="link_3" />
+        <origin xyz="0.225 0 0" rpy="0 0 0" />
+        <axis xyz="0 0 1" />
+        <limit effort="1000.0" velocity="100.0"
+            lower="-2.51" upper="2.51" />
+    </joint>
+    <joint name="joint_4" type="revolute">
+        <parent link="link_3" />
+        <child link="link_4" />
+        <origin xyz="0.2 0 0" rpy="0 0 0" />
+        <axis xyz="0 0 1" />
+        <limit effort="1000.0" velocity="100.0"
+            lower="-2.51" upper="2.51" />
+    </joint>
+    <joint name="joint_5" type="revolute">
+        <parent link="link_4" />
+        <child link="link_5" />
+        <origin xyz="0.0915 0 0" rpy="0 1.57 0" />
+        <axis xyz="0 0 1" />
+        <limit effort="1000.0" velocity="100.0"
+            lower="-2.51" upper="2.51" />
+    </joint>
+    <joint name="joint_6" type="prismatic">
+        <parent link="link_5" />
+        <child link="gripper_right" />
+        <origin xyz="-0.01 0 0.1015" rpy="0 0 0" />
+        <axis xyz="0 1 0" />
+        <limit effort="1000.0" velocity="100.0"
+            lower="-0.018" upper="0.02" />
+    </joint>
+    <joint name="joint_7" type="prismatic">
+        <parent link="link_5" />
+        <child link="gripper_left" />
+        <origin xyz="-0.01 0 0.1015" rpy="0 0 0" />
+        <axis xyz="0 1 0" />
+        <mimic joint="joint_6" multiplier="-1" />
+        <limit effort="1000.0" velocity="100.0"
+            lower="-0.018" upper="0.02" />
+    </joint>
 </robot>

File: install/robot_description/share/robot_description/urdf/skyentific_robot_ros2_control.xacro (robot description, xacro)
@@ -2,8 +2,11 @@
 <robot xmlns:xacro="http://www.ros.org/wiki/xacro">
     <ros2_control name="Arm" type="system">
+        ...
+</ros2_control>
+    <ros2_control name="Gripper" type="system">
         <hardware>
             <plugin>mock_components/GenericSystem</plugin>
         </hardware>
-        <joint name="joint_1">
+        <joint name="joint_6">
             <command_interface name="position" />
             <state_interface name="position">

Commit message: Remove deprecated setup scripts and related files for robot_moveit_config package
- Deleted local_setup.zsh, package.bash, package.dsv, package.ps1, package.sh, package.xml, package.zsh, and setup scripts (bash, ps1, sh, zsh) as they are no longer needed.
- Removed compiled Python files from the launch directory.
- Cleaned up the installation structure by eliminating unnecessary files to streamline the package.

File: install/robot_description/share/robot_description/urdf/skyentific_robot.urdf.xacro (robot description, xacro)
@@ -1,208 +1 @@
-<?xml version="1.0"?>
-<robot name="skyentific_robot"
-    xmlns:xacro="http://www.ros.org/wiki/xacro">
-    <!-- Include ros2_control Plugins -->
-    <xacro:include filename="$(find robot_description)/urdf/skyentific_robot_ros2_control.xacro" />
-    <!-- Useful XACRO Variables (Properties) -->
-    <xacro:property name="PI" value="3.14159265359" />
-    <material name="grey">
-        <color rgba="0.5 0.5 0.5 1.0" />
-    </material>
-    <material name="red">
-        <color rgba="0.5 0.0 0.0 1.0" />
-    </material>
-    <link name="base_link">
-        <visual>
-            <origin xyz="0 0 0" rpy="0 0 0" />
-            <geometry>
-                <mesh filename="file://$(find robot_description)/meshes/base_z_ob.stl"
-                    scale="0.001 0.001 0.001" />
-            </geometry>
-            <material name="grey" />
-        </visual>
-        <collision> <!-- cyclinder equivalent -->
-            <origin xyz="0 0 0.075" rpy="0 0 0" />
-            <geometry>
-                <cylinder radius="0.1" length="0.15" />
-            </geometry>
-        </collision>
-    </link>
-    <link name="link_1">
-        <visual>
-            <origin xyz="0 0 0" rpy="0 0 0" />
-            <geometry>
-                <mesh filename="file://$(find robot_description)/meshes/link_1.stl"
-                    scale="0.001 0.001 0.001" />
-            </geometry>
-            <material name="grey" />
-        </visual>
-        <collision>
-            <origin xyz="0 0 0.150" rpy="1.57 0 0" />
-            <geometry>
-                <cylinder radius="0.095" length="0.1" />
-            </geometry>
-        </collision>
-    </link>
-    <link name="link_2">
-        <visual>
-            <origin xyz="0 0 0" rpy="0 0 0" />
-            <geometry>
-                <mesh filename="file://$(find robot_description)/meshes/link_2.stl"
-                    scale="0.001 0.001 0.001" />
-            </geometry>
-            <material name="grey" />
-        </visual>
-        <collision>
-            <origin xyz="0.225 0 0 " rpy="0 0 0" />
-            <geometry>
-                <cylinder radius="0.07" length="0.1" />
-            </geometry>
-        </collision>
-    </link>
-    <link name="link_3">
-        <visual>
-            <origin xyz="0 0 0" rpy="0 0 0" />
-            <geometry>
-                <mesh filename="file://$(find
-robot_description)/meshes/link_3.stl"
-                    scale="0.001 0.001 0.001" />
-            </geometry>
-            <material name="grey" />
-        </visual>
-        <collision>
-            <origin xyz="0.2 0 0" rpy="0 0 0" />
-            <geometry>
-                <cylinder radius="0.055" length="0.1" />
-            </geometry>
-        </collision>
-    </link>
-    <link name="link_4">
-        <visual>
-            <origin xyz="0 0 0" rpy="0 0 0" />
-            <geometry>
-                <mesh filename="file://$(find
-robot_description)/meshes/link_4.stl"
-                    scale="0.001 0.001 0.001" />
-            </geometry>
-            <material name="grey" />
-        </visual>
-        <collision>
-            <origin xyz="0.1 0 0" rpy="0 1.57 0" />
-            <geometry>
-                <cylinder radius="0.055"
-                    length="0.06" />
-            </geometry>
-        </collision>
-    </link>
-    <link name="link_5">
-        <visual>
-            <origin xyz="0 0 0" rpy="0 0 0" />
-            <geometry>
-                <mesh filename="file://$(find
-robot_description)/meshes/link_5_gripper.stl"
-                    scale="0.001 0.001 0.001" />
-            </geometry>
-            <material name="grey" />
-        </visual>
-        <collision>
-            <origin xyz="0 0 0" rpy="1.57 0 0" />
-            <geometry>
-                <cylinder radius="0.055"
-                    length="0.01" />
-            </geometry>
-        </collision>
-    </link>
-    <link name="gripper_right">
-        <visual>
-            <origin xyz="0 0 0" rpy="0 0 0" />
-            <geometry>
-                <mesh filename="file://$(find
-robot_description)/meshes/rightjaw.stl"
-                    scale="0.001 0.001 0.001" />
-            </geometry>
-            <material name="red" />
-        </visual>
-        <collision>
-            <origin xyz="0.01 0.025 0.045" rpy="0 0 0" />
-            <geometry>
-                <cylinder radius="0.0125"
-                    length="0.04" />
-            </geometry>
-        </collision>
-    </link>
-    <link name="gripper_left">
-        <visual>
-            <origin xyz="0 0 0" rpy="0 0 0" />
-            <geometry>
-                <mesh filename="file://$(find
-robot_description)/meshes/leftjaw.stl"
-                    scale="0.001 0.001 0.001" />
-            </geometry>
-            <material name="red" />
-        </visual>
-        <collision>
-            <origin xyz="0.01 -0.025 0.045" rpy="0 0 0" />
-            <geometry>
-                <cylinder radius="0.0125"
-                    length="0.04" />
-            </geometry>
-        </collision>
-    </link>
-    <joint name="joint_1" type="revolute">
-        <parent link="base_link" />
-        <child link="link_1" />
-        <origin xyz="0 0 0.0965" rpy="0 0 0" />
-        <axis xyz="0 0 1" />
-        <limit effort="1000.0" velocity="100.0"
-            lower="-3.14" upper="3.14" />
-    </joint>
-    <joint name="joint_2" type="revolute">
-        <parent link="link_1" />
-        <child link="link_2" />
-        <origin xyz="0 0 0.150" rpy="0 -1.57 1.57 " />
-        <axis xyz="0 0 1" />
-        <limit effort="1000.0" velocity="100.0"
-            lower="-2.51" upper="2.51" />
-    </joint>
-    <joint name="joint_3" type="revolute">
-        <parent link="link_2" />
-        <child link="link_3" />
-        <origin xyz="0.225 0 0" rpy="0 0 0" />
-        <axis xyz="0 0 1" />
-        <limit effort="1000.0" velocity="100.0"
-            lower="-2.51" upper="2.51" />
-    </joint>
-    <joint name="joint_4" type="revolute">
-        <parent link="link_3" />
-        <child link="link_4" />
-        <origin xyz="0.2 0 0" rpy="0 0 0" />
-        <axis xyz="0 0 1" />
-        <limit effort="1000.0" velocity="100.0"
-            lower="-2.51" upper="2.51" />
-    </joint>
-    <joint name="joint_5" type="revolute">
-        <parent link="link_4" />
-        <child link="link_5" />
-        <origin xyz="0.0915 0 0" rpy="0 1.57 0" />
-        <axis xyz="0 0 1" />
-        <limit effort="1000.0" velocity="100.0"
-            lower="-2.51" upper="2.51" />
-    </joint>
-    <joint name="joint_6" type="prismatic">
-        <parent link="link_5" />
-        <child link="gripper_right" />
-        <origin xyz="-0.01 0 0.1015" rpy="0 0 0" />
-        <axis xyz="0 1 0" />
-        <limit effort="1000.0" velocity="100.0"
-            lower="-0.018" upper="0.02" />
-    </joint>
-    <joint name="joint_7" type="prismatic">
-        <parent link="link_5" />
-        <child link="gripper_left" />
-        <origin xyz="-0.01 0 0.1015" rpy="0 0 0" />
-        <axis xyz="0 1 0" />
-        <mimic joint="joint_6" multiplier="-1" />
-        <limit effort="1000.0" velocity="100.0"
-            lower="-0.018" upper="0.02" />
-    </joint>
-</robot>
+/home/tyrhaton/Projects/les_ws/src/robot_description/urdf/skyentific_robot.urdf.xacro

File: install/robot_description/share/robot_description/urdf/skyentific_robot_ros2_control.xacro (robot description, xacro)
@@ -1,17 +1 @@
-<?xml version="1.0"?>
-<robot xmlns:xacro="http://www.ros.org/wiki/xacro">
-    <ros2_control name="Arm" type="system">
-        ...
-</ros2_control>
-    <ros2_control name="Gripper" type="system">
-        <hardware>
-            <plugin>mock_components/GenericSystem</plugin>
-        </hardware>
-        <joint name="joint_6">
-            <command_interface name="position" />
-            <state_interface name="position">
-                <param name="initial_value">0.0</param>
-            </state_interface>
-        </joint>
-    </ros2_control>
-</robot>
+/home/tyrhaton/Projects/les_ws/src/robot_description/urdf/skyentific_robot_ros2_control.xacro

File: install/robot_moveit_config/share/robot_moveit_config/config/skyentific_robot.ros2_control.xacro (robot description, xacro)
@@ -1,48 +1 @@
-<?xml version="1.0"?>
-<robot xmlns:xacro="http://www.ros.org/wiki/xacro">
-    <xacro:macro name="skyentific_robot_ros2_control" params="name initial_positions_file">
-        <xacro:property name="initial_positions" value="${xacro.load_yaml(initial_positions_file)['initial_positions']}"/>
-        <ros2_control name="${name}" type="system">
-            <hardware>
-                <!-- By default, set up controllers for simulation. This won't work on real hardware -->
-                <plugin>mock_components/GenericSystem</plugin>
-            </hardware>
-            <joint name="joint_1">
-                <command_interface name="position"/>
-                <state_interface name="position">
-                  <param name="initial_value">${initial_positions['joint_1']}</param>
-                </state_interface>
-            </joint>
-            <joint name="joint_2">
-                <command_interface name="position"/>
-                <state_interface name="position">
-                  <param name="initial_value">${initial_positions['joint_2']}</param>
-                </state_interface>
-            </joint>
-            <joint name="joint_3">
-                <command_interface name="position"/>
-                <state_interface name="position">
-                  <param name="initial_value">${initial_positions['joint_3']}</param>
-                </state_interface>
-            </joint>
-            <joint name="joint_4">
-                <command_interface name="position"/>
-                <state_interface name="position">
-                  <param name="initial_value">${initial_positions['joint_4']}</param>
-                </state_interface>
-            </joint>
-            <joint name="joint_5">
-                <command_interface name="position"/>
-                <state_interface name="position">
-                  <param name="initial_value">${initial_positions['joint_5']}</param>
-                </state_interface>
-            </joint>
-            <joint name="joint_6">
-                <command_interface name="position"/>
-                <state_interface name="position">
-                  <param name="initial_value">${initial_positions['joint_6']}</param>
-                </state_interface>
-            </joint>
-        </ros2_control>
-    </xacro:macro>
-</robot>
+/home/tyrhaton/Projects/les_ws/src/robot_moveit_config/config/skyentific_robot.ros2_control.xacro

File: install/robot_moveit_config/share/robot_moveit_config/config/skyentific_robot.urdf.xacro (robot description, xacro)
@@ -1,9 +1 @@
-<?xml version="1.0"?>
-<robot xmlns:xacro="http://www.ros.org/wiki/xacro" name="skyentific_robot">
-    <xacro:arg name="initial_positions_file" default="initial_positions.yaml" />
-    <!-- Import skyentific_robot urdf file -->
-    <xacro:include filename="$(find robot_description)/urdf/skyentific_robot.urdf.xacro" />
-    <!-- Import control_xacro -->
-    <xacro:include filename="skyentific_robot.ros2_control.xacro" />
-    <xacro:skyentific_robot_ros2_control name="FakeSystem" initial_positions_file="$(arg initial_positions_file)"/>
-</robot>
+/home/tyrhaton/Projects/les_ws/src/robot_moveit_config/config/skyentific_robot.urdf.xacro

File: src/robot_description/urdf/skyentific_robot_ros2_control.xacro (robot description, xacro)
@@ -1,17 +1,70 @@
 <?xml version="1.0"?>
 <robot xmlns:xacro="http://www.ros.org/wiki/xacro">
+  <xacro:arg name="use_mock_component" default="true"/>
+  <xacro:arg name="use_moveit_control" default="false"/>
+  <!-- Only include this ros2_control block when not using MoveIt (which has its own) -->
+  <xacro:unless value="$(arg use_moveit_control)">
     <ros2_control name="Arm" type="system">
-        ...
-</ros2_control>
+      <hardware>
+        <xacro:if value="$(arg use_mock_component)">
+          <plugin>mock_components/GenericSystem</plugin>
+        </xacro:if>
+        <xacro:unless value="$(arg use_mock_component)">
+          <plugin>arm_hardware/ArmHardwareInterface</plugin>
+          <param name="port">/dev/ttyACM0</param>
+          <param name="baudrate">57600</param>
+          <param name="motor_id_1">1</param>
+          <param name="motor_id_2">2</param>
+          <param name="motor_id_3">3</param>
+          <param name="motor_id_4">4</param>
+          <param name="motor_id_5">5</param>
+          <param name="steps_per_rev">200.0</param>
+          <param name="hex_dump">false</param>
+          <param name="probe">false</param>
+          <param name="protocol">register</param>
+        </xacro:unless>
+      </hardware>
+      <joint name="joint_1">
+        <command_interface name="position"/>
+        <state_interface name="position">
+          <param name="initial_value">0.0</param>
+        </state_interface>
+      </joint>
+      <joint name="joint_2">
+        <command_interface name="position"/>
+        <state_interface name="position">
+          <param name="initial_value">0.0</param>
+        </state_interface>
+      </joint>
+      <joint name="joint_3">
+        <command_interface name="position"/>
+        <state_interface name="position">
+          <param name="initial_value">0.0</param>
+        </state_interface>
+      </joint>
+      <joint name="joint_4">
+        <command_interface name="position"/>
+        <state_interface name="position">
+          <param name="initial_value">0.0</param>
+        </state_interface>
+      </joint>
+      <joint name="joint_5">
+        <command_interface name="position"/>
+        <state_interface name="position">
+          <param name="initial_value">0.0</param>
+        </state_interface>
+      </joint>
+    </ros2_control>
     <ros2_control name="Gripper" type="system">
-        <hardware>
-            <plugin>mock_components/GenericSystem</plugin>
-        </hardware>
-        <joint name="joint_6">
-            <command_interface name="position" />
-            <state_interface name="position">
-                <param name="initial_value">0.0</param>
-            </state_interface>
-        </joint>
+      <hardware>
+        <plugin>mock_components/GenericSystem</plugin>
+      </hardware>
+      <joint name="joint_6">
+        <command_interface name="position" />
+        <state_interface name="position">
+          <param name="initial_value">0.0</param>
+        </state_interface>
+      </joint>
     </ros2_control>
+  </xacro:unless>
 </robot>
